File: PCB/Matyas's Hackpad.kicad_pcb (KiCad board)
At the start: 2 copper layers, 80 x 62.5 mm, 27 parts, among them J1 OLED_DISPLAY, SW1 SW_Push, SW2 SW_Push, SW3 SW_Push, SW4 RotaryEncoder_Switch, SW5 SW_Push, SW6 SW_Push, SW7 SW_Push, SW8 SW_Push, U1 MOUDLE-SEEEDUINO-XIAO

Commit message: Fix
Routing:
- net GND: track 211.2 -> 210.7 mm
Changed lines of the file:
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@@
-	)
-	(segment
-		(start 182.37 87.802)
-		(end 181.181 88.991)
-		(width 0.2)
-		(layer "B.Cu")
-		(net 13)
 	)
 	(segment
@@
 	)
 	(segment
-		(start 181.181 88.991)
+		(start 182.37 86.94)
+		(end 185.07 89.64)
+		(width 0.2)
+		(layer "B.Cu")
+		(net 13)
+	)
+	(segment
+		(start 156.375 87.84)
 		(end 157.526 88.991)
 		(width 0.2)
@@
 	)
 	(segment
+		(start 180.199 88.991)
+		(end 182.25 86.94)
+		(width 0.2)
+		(layer "B.Cu")
+		(net 13)
+	)
+	(segment
 		(start 183.3 116.3)
 		(end 183.3 120.75)
@@
 	)
 	(segment
-		(start 182.37 86.94)
-		(end 182.37 87.802)
-		(width 0.2)
-		(layer "B.Cu")
-		(net 13)
-	)
-	(segment
 		(start 138.050001 138.872158)
 		(end 140.652843 141.475)
@@
 	)
 	(segment
-		(start 157.526 88.991)
-		(end 156.375 87.84)
-		(width 0.2)
-		(layer "B.Cu")
-		(net 13)
-	)
-	(segment
 		(start 179.827842 119.772158)
 		(end 176.150001 119.772158)
@@
 	)
 	(segment
-		(start 185.07 89.64)
+		(start 157.526 88.991)
+		(end 180.199 88.991)
+		(width 0.2)
+		(layer "B.Cu")
+		(net 13)
+	)
+	(segment
+		(start 182.25 86.94)
 		(end 182.37 86.94)
 		(width 0.2)
@@
 	)
 	(segment
+		(start 181.145 88.375)
+		(end 179.375 88.375)
+		(width 0.2)
+		(layer "F.Cu")
+		(net 14)
+	)
+	(segment
 		(start 142.9 113)
 		(end 148.2 118.3)
@@
 	)
 	(segment
-		(start 179.375 88.375)
-		(end 181.265 88.375)
-		(width 0.2)
-		(layer "F.Cu")
-		(net 14)
-	)
-	(segment
-		(start 181.265 88.375)
-		(end 182.37 89.48)
-		(width 0.2)
-		(layer "F.Cu")
+		(start 182.25 89.48)
+		(end 181.145 88.375)
+		(width 0.2)
+		(layer "F.Cu")

Commit message: Fix for manufacture
Other:
- board text added: "DESIGN MADE IN CZECHIA"
- board text removed: "MADE IN CZECHIA"
Changed lines of the file:
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@@
 			(drillshape 0)
 			(scaleselection 1)
-			(outputdirectory "")
+			(outputdirectory "C:/Users/já/Downloads/")
 		)
 	)
@@
 		)
 	)
-	(gr_text "MADE IN CZECHIA"
+	(gr_text "DESIGN MADE IN CZECHIA"
 		(at 202.15 142.9 0)
 		(layer "B.SilkS")
